Commit message: Fix package://meshes in kuka_description

File: skrobot/data/kuka_description/kuka.urdf (robot description, URDF)
Before this commit: robot lbr_iiwa_with_wsg50, 15 links, 14 joints
Links:
- link lbr_iiwa_with_wsg50__lbr_iiwa_link_0: geometry collision mesh filename=meshes/link_0.stl scale=1 1 1; visual mesh filename=meshes/link_0.stl scale=1 1 1
- link lbr_iiwa_with_wsg50__lbr_iiwa_link_1: geometry collision mesh filename=meshes/link_1.stl scale=1 1 1; visual mesh filename=meshes/link_1.stl scale=1 1 1
- link lbr_iiwa_with_wsg50__lbr_iiwa_link_2: geometry collision mesh filename=meshes/link_2.stl scale=1 1 1; visual mesh filename=meshes/link_2.stl scale=1 1 1
- link lbr_iiwa_with_wsg50__lbr_iiwa_link_3: geometry collision mesh filename=meshes/link_3.stl scale=1 1 1; visual mesh filename=meshes/link_3.stl scale=1 1 1
- link lbr_iiwa_with_wsg50__lbr_iiwa_link_4: geometry collision mesh filename=meshes/link_4.stl scale=1 1 1; visual mesh filename=meshes/link_4.stl scale=1 1 1
- link lbr_iiwa_with_wsg50__lbr_iiwa_link_5: geometry collision mesh filename=meshes/link_5.stl scale=1 1 1; visual mesh filename=meshes/link_5.stl scale=1 1 1
- link lbr_iiwa_with_wsg50__lbr_iiwa_link_6: geometry collision mesh filename=meshes/link_6.stl scale=1 1 1; visual mesh filename=meshes/link_6.stl scale=1 1 1
- link lbr_iiwa_with_wsg50__lbr_iiwa_link_7: geometry collision mesh filename=meshes/link_7.stl scale=1 1 1; visual mesh filename=meshes/link_7.stl scale=1 1 1
- link lbr_iiwa_with_wsg50__left_finger_base: geometry collision mesh filename=meshes/finger_base_left.stl scale=1 1 1; visual mesh filename=meshes/finger_base_left.stl scale=1 1 1
- link lbr_iiwa_with_wsg50__left_finger_tip: geometry collision mesh filename=meshes/finger_tip_left.stl scale=1 1 1; visual mesh filename=meshes/finger_tip_left.stl scale=1 1 1
- link lbr_iiwa_with_wsg50__right_finger_base: geometry collision mesh filename=meshes/finger_base_right.stl scale=1 1 1; visual mesh filename=meshes/finger_base_right.stl scale=1 1 1
- link lbr_iiwa_with_wsg50__right_finger_tip: geometry collision mesh filename=meshes/finger_tip_right.stl scale=1 1 1; visual mesh filename=meshes/finger_tip_right.stl scale=1 1 1

Commit message: Add max joint velocity for kuka and pr2

File: skrobot/data/kuka_description/kuka.urdf (robot description, URDF)
Before this commit: robot lbr_iiwa_with_wsg50, 15 links, 14 joints
Joints:
- joint lbr_iiwa_with_wsg50__base_left_finger_joint: limit lower=-10.4 upper=10.01 effort=100.0 velocity=0.0 -> lower=-10.4 upper=10.01 effort=100.0 velocity=1.0
- joint lbr_iiwa_with_wsg50__base_right_finger_joint: limit lower=-10.01 upper=10.4 effort=100.0 velocity=0.0 -> lower=-10.01 upper=10.4 effort=100.0 velocity=1.0
- joint lbr_iiwa_with_wsg50__gripper_to_arm: type continuous -> fixed
- joint lbr_iiwa_with_wsg50__left_base_tip_joint: limit lower=-10.1 upper=10.3 effort=0.0 velocity=0.0 -> lower=-10.1 upper=10.3 effort=0.0 velocity=1.0
- joint lbr_iiwa_with_wsg50__right_base_tip_joint: limit lower=-10.3 upper=10.1 effort=0.0 velocity=0.0 -> lower=-10.3 upper=10.1 effort=0.0 velocity=1.0
